Commit message: Return to diff_drive

File: m5/ex03/src/robot_description/urdf/car.xacro (robot description, xacro)
@@ -1,38 +1,18 @@
 <?xml version="1.0"?>
 <robot name='robot' xmlns:xacro="http://ros.org/wiki/xacro">
-  <!-- Define wheel radius, suspension parameters, and car dimensions -->
-  <!-- kingpin_width = chassis_width + suspension_joint_with_chassis_offset_y * 2 -->
-  <!-- wheel_separation = chassis_width + suspension_joint_with_chassis_offset_y * 2 + (steering_radius - wheel_width / 2) * 2 -->
   <xacro:property name="wheel_offset_x" value="0.226"/>
   <xacro:property name="wheel_offset_y" value="0.1485"/>
-  <xacro:property name="wheel_offset_z" value="-0.2"/>
+  <xacro:property name="wheel_offset_z" value="-1.0"/>
   <xacro:property name="wheel_radius" value="0.2"/>
   <xacro:property name="wheel_width" value="0.1"/>
-  <xacro:property name="suspension_length" value="0.2"/>
-  <xacro:property name="suspension_radius" value="0.1"/>
-  <xacro:property name="chassis_height" value="0.5"/>
-  <xacro:property name="chassis_width" value="0.8"/>
-  <xacro:property name="chassis_length" value="1.6"/>
+  <xacro:property name="body_height" value="0.2"/>
+  <xacro:property name="body_width" value="0.8"/>
+  <xacro:property name="body_length" value="1.6"/>
+  <xacro:property name="wheeltrack" value="1.5"/>
   <xacro:property name="wheelbase" value="1.5"/>
-  <xacro:property name="steering_radius" value="0.2"/>
-  <xacro:property name="suspension_joint_with_chassis_offset_z" value="0.0"/>
-  <xacro:property name="suspension_joint_with_chassis_offset_y" value="0.0"/>
-  <xacro:property name="suspension_joint_with_chassis_offset_x" value="0.0"/>
+  <xacro:property name="chassis_offset_z" value="0.2"/>
+  <xacro:property name="chassis_offset_y" value="0.0"/>
+  <xacro:property name="chassis_offset_x" value="0.0"/>
   <xacro:include filename="$(find robot_description)/urdf/gazebo.urdf.xacro" />
-  <material name="white">
-      <color rgba="1 1 1 1" />
-  </material>
-  <material name="orange">
-      <color rgba="1 0.3 0.1 1"/>
-  </material>
-  <material name="blue">
-      <color rgba="0.2 0.2 1 1"/>
-  </material>
-  <material name="black">
-      <color rgba="0 0 0 1"/>
-  </material>
-  <material name="red">
-      <color rgba="1 0 0 1"/>
-  </material>
   <link name="base_link">
   </link>
@@ -40,57 +20,28 @@
   </link>
   <joint name="base_footprint_joint" type="fixed">
-      <parent link="base_link"/>
-      <child link="base_footprint"/>
-      <origin xyz="0 0 -0.138" rpy="0 0 0"/>
+    <parent link="base_link"/>
+    <child link="base_footprint"/>
+    <origin rpy="0 0 0" xyz="0 0 -0.138"/>
   </joint>
-  <joint name="chassis_joint" type="fixed">
-      <parent link="base_link"/>
-      <child link="chassis_link"/>
-      <origin xyz="${-wheel_offset_x} 0 ${-wheel_offset_z}"/>
+  <joint name="body_joint" type="fixed">
+    <parent link="base_link"/>
+    <child link="body_link"/>
+    <origin xyz="${-wheel_offset_x} 0 ${-wheel_offset_z}"/>
   </joint>
-  <!-- Car body -->
-  <link name="chassis_link">
+  <link name="body_link">
     <visual>
       <geometry>
-        <box size="${chassis_length} ${chassis_width} ${chassis_height}"/>
+        <box size="${body_length} ${body_width} ${body_height}"/>
       </geometry>
     </visual>
     <collision>
       <geometry>
-        <box size="${chassis_length} ${chassis_width} ${chassis_height}"/>
+        <box size="${body_length} ${body_width} ${body_height}"/>
       </geometry>
     </collision>
   </link>
-  <gazebo reference="chassis">
-        <material>Gazebo/Blue</material>
+  <gazebo reference="body">
+    <material>Gazebo/Blue</material>
   </gazebo>
-  <!-- Front left wheel -->
-  <joint name="front_left_steering_joint" type="revolute">
-    <origin xyz="${wheelbase / 2 + suspension_joint_with_chassis_offset_x} ${chassis_width / 2 + suspension_joint_with_chassis_offset_y} -${suspension_joint_with_chassis_offset_z}"/>
-    <parent link="chassis_link"/>
-    <child link="front_left_suspension_link"/>
-    <axis xyz="0 0 1"/>
-    <limit effort="100" velocity="1.0"/>
-  </joint>
-  <!-- Front right wheel -->
-  <joint name="front_right_steering_joint" type="revolute">
-    <origin xyz="${wheelbase / 2 + suspension_joint_with_chassis_offset_x} -${chassis_width / 2 + suspension_joint_with_chassis_offset_y} -${suspension_joint_with_chassis_offset_z}"/>
-    <parent link="chassis_link"/>
-    <child link="front_right_suspension_link"/>
-    <axis xyz="0 0 1"/>
-    <limit effort="100" velocity="1.0"/>
-  </joint>
-  <!-- Rear left wheel -->
-  <joint name="rear_left_chassis_joint" type="fixed">
-    <origin xyz="-${wheelbase / 2 - suspension_joint_with_chassis_offset_x} ${chassis_width / 2 + suspension_joint_with_chassis_offset_y} -${suspension_joint_with_chassis_offset_z}"/>
-    <parent link="chassis_link"/>
-    <child link="rear_left_suspension_link"/>
-  </joint>
-  <!-- Rear ight wheel -->
-  <joint name="rear_right_chassis_joint" type="fixed">
-    <origin xyz="-${wheelbase / 2 - suspension_joint_with_chassis_offset_x} -${chassis_width / 2 + suspension_joint_with_chassis_offset_y} -${suspension_joint_with_chassis_offset_z}"/>
-    <parent link="chassis_link"/>
-    <child link="rear_right_suspension_link"/>
-  </joint>
   <xacro:macro name="wheel" params="prefix">
     <link name="${prefix}_wheel_link">
@@ -113,5 +64,5 @@
       </inertial>
     </link>
-    <gazebo reference="${prefix}_wheel">
+    <gazebo reference="${prefix}_wheel_link">
         <material>Gazebo/Blue</material>
     </gazebo>
@@ -121,81 +72,15 @@
   <xacro:wheel prefix="rear_left"/>
   <xacro:wheel prefix="rear_right"/>
-  <xacro:macro name="suspension" params="prefix">
-    <link name="${prefix}_suspension_link">
-      <visual>
-        <geometry>
-          <cylinder length="${suspension_length}" radius="${suspension_radius}"/>
-        </geometry>
-      </visual>
-      <collision>
-        <geometry>
-          <cylinder length="${suspension_length}" radius="${suspension_radius}"/>
-        </geometry>
-      </collision>
-      <inertial>
-        <origin xyz="0 0 0"/>
-        <mass value="0.5"/>
-        <inertia ixx="0.01" ixy="0.0" ixz="0.0" iyy="0.01" iyz="0.0" izz="0.01"/>
-      </inertial>
-    </link>
-    <gazebo reference="${prefix}_suspension">
-        <material>Gazebo/Blue</material>
-    </gazebo>
-  </xacro:macro>
-  <xacro:suspension prefix="front_left"/>
-  <xacro:suspension prefix="front_right"/>
-  <xacro:suspension prefix="rear_left"/>
-  <xacro:suspension prefix="rear_right"/>
-  <xacro:macro name="hub" params="prefix">
-    <link name="${prefix}_hub_link">
-      <visual>
-        <geometry>
-          <sphere radius="0.01"/>
-        </geometry>
-      </visual>
-      <collision>
-        <geometry>
-          <sphere radius="0.01"/>
-        </geometry>
-      </collision>
-      <inertial>
-        <origin xyz="0 0 0"/>
-        <mass value="1.0"/>
-        <inertia ixx="0.01" ixy="0.0" ixz="0.0" iyy="0.01" iyz="0.0" izz="0.01"/>
-      </inertial>
-    </link>
-    <gazebo reference="${prefix}_hub">
-        <material>Gazebo/Blue</material>
-    </gazebo>
-  </xacro:macro>
-  <xacro:hub prefix="front_left"/>
-  <xacro:hub prefix="front_right"/>
-  <xacro:hub prefix="rear_left"/>
-  <xacro:hub prefix="rear_right"/>
-  <xacro:macro name="suspension_with_hub_joint" params="prefix origin_xyz">
-    <joint name="${prefix}_suspension_with_hub_joint" type="prismatic">
+  <xacro:macro name="wheel_joint" params="prefix origin_xyz">
+    <joint name="${prefix}_wheel_joint" type="continuous">
       <origin xyz="${origin_xyz}"/>
-      <parent link="${prefix}_suspension_link"/>
-      <child link="${prefix}_hub_link"/>
-      <axis xyz="0 0 1"/>
-      <limit effort="100" velocity="1.0" lower="-${suspension_length}" upper="0.0"/>
-      <dynamics damping="0.7"/>
-    </joint>
-  </xacro:macro>
-  <xacro:suspension_with_hub_joint prefix="front_left" origin_xyz="0 ${steering_radius} 0"/>
-  <xacro:suspension_with_hub_joint prefix="front_right" origin_xyz="0 -${steering_radius} 0"/>
-  <xacro:suspension_with_hub_joint prefix="rear_left" origin_xyz="0 ${steering_radius} 0"/>
-  <xacro:suspension_with_hub_joint prefix="rear_right" origin_xyz="0 -${steering_radius} 0"/>
-  <xacro:macro name="hub_with_wheel_joint" params="prefix">
-    <joint name="${prefix}_hub_with_wheel_joint" type="continuous">
-      <origin xyz="0 0 0"/>
-      <parent link="${prefix}_hub_link"/>
+      <parent link="base_link"/>
       <child link="${prefix}_wheel_link"/>
       <axis xyz="0 1 0"/>
     </joint>
   </xacro:macro>
-  <xacro:hub_with_wheel_joint prefix="front_left"/>
-  <xacro:hub_with_wheel_joint prefix="front_right"/>
-  <xacro:hub_with_wheel_joint prefix="rear_left"/>
-  <xacro:hub_with_wheel_joint prefix="rear_right"/>
+  <xacro:wheel_joint prefix="front_left" origin_xyz="${wheelbase / 2 + chassis_offset_x} ${wheeltrack / 2 + chassis_offset_y} ${chassis_offset_z}"/>
+  <xacro:wheel_joint prefix="front_right" origin_xyz="${wheelbase / 2 + chassis_offset_x} ${-wheeltrack / 2 + chassis_offset_y} ${chassis_offset_z}"/>
+  <xacro:wheel_joint prefix="rear_left" origin_xyz="${-wheelbase / 2 + chassis_offset_x} ${wheeltrack / 2 + chassis_offset_y} ${chassis_offset_z}"/>
+  <xacro:wheel_joint prefix="rear_right" origin_xyz="${-wheelbase / 2 + chassis_offset_x} ${-wheeltrack / 2 + chassis_offset_y} ${chassis_offset_z}"/>
 </robot>

File: m5/ex03/src/robot_description/urdf/gazebo.urdf.xacro (robot description, xacro)
@@ -17,26 +17,17 @@
             <odom_publish_frequency>50</odom_publish_frequency>
         </plugin-->
-        <!-- <plugin
+        <plugin
             filename="gz-sim-joint-state-publisher-system"
             name="gz::sim::systems::JointStatePublisher">
-        </plugin> -->
+        </plugin>
         <plugin
-            filename="libgz-sim7-ackermann-steering-system.so"
-            name="gz::sim::v7::systems::AckermannSteering">
-            <steering_only>false</steering_only>
-            <!-- <use_actuator_msg></use_actuator_msg>
-            <actuator_number></actuator_number> -->
-            <!-- <steer_p_gain></steer_p_gain> -->
-            <left_steering_joint>front_left_steering_joint</left_steering_joint>
-            <right_steering_joint>front_right_steering_joint</right_steering_joint>
-            <left_joint>front_left_hub_with_wheel_joint</left_joint>
-            <right_joint>front_right_hub_with_wheel_joint</right_joint>
-            <left_joint>rear_left_hub_with_wheel_joint</left_joint>
-            <right_joint>rear_right_hub_with_wheel_joint</right_joint>
-            <wheel_separation>${chassis_width + suspension_joint_with_chassis_offset_y * 2 + (steering_radius - wheel_width / 2) * 2}</wheel_separation>
-            <kingpin_width>${chassis_width + suspension_joint_with_chassis_offset_y * 2}</kingpin_width>
-            <wheel_base>${chassis_width + suspension_joint_with_chassis_offset_y * 2 + steering_radius * 2}</wheel_base>
-            <steering_limit>0.5</steering_limit>
-            <wheel_radius>${wheel_radius}</wheel_radius>
+            filename="gz-sim-diff-drive-system"
+            name="gz::sim::systems::DiffDrive">
+            <left_joint>left_wheel_joint</left_joint>
+            <right_joint>right_wheel_joint</right_joint>
+            <child_frame_id>robot/base_link</child_frame_id>
+            <wheel_separation>0.291</wheel_separation>
+            <wheel_radius>0.033</wheel_radius>
+            <odom_publish_frequency>10</odom_publish_frequency>
         </plugin>
     </gazebo>
